File: H1DR0/design/H1DR00.brd (EAGLE design)
At the start: 34.6 x 30 mm, 33 parts, among them IC2 MAX3232CSE, P1 HEXABIT_17.32_NO_P6, U1 STM32F091CBU6, X1 XTALL_CSTCE8M00G52

Commit message: OUTPUT CAM  files generated
Changed lines of the file:
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@@
 <?xml version="1.0" encoding="utf-8"?>
 <!DOCTYPE eagle SYSTEM "eagle.dtd">
-<eagle version="9.6.0">
+<eagle version="9.6.1">
 <drawing>
 <settings>
@@
 </element>
 <element name="IC2" library="Hexabitz" package="SO16" package3d_urn="urn:adsk.eagle:package:821/2" value="MAX3232CSE" x="34.671" y="34.671" smashed="yes" rot="R90">
+<attribute name="DESCRIPTION" value="MAX3232 Series 235 kbps 5.5 V Surface Mount RS-232 Transceiver - SOIC-16" x="34.671" y="34.671" size="1.778" layer="27" rot="R90" display="off"/>
 <attribute name="MF" value="" x="34.671" y="34.671" size="1.778" layer="27" rot="R90" display="off"/>
+<attribute name="MFN" value="Maxim Integrated" x="34.671" y="34.671" size="1.778" layer="27" rot="R90" display="off"/>
 <attribute name="MPN" value="MAX3232CSE" x="34.671" y="34.671" size="1.778" layer="27" rot="R90" display="off"/>
 <attribute name="NAME" x="34.925" y="29.21" size="1.27" layer="25" ratio="10" rot="R180"/>
+<attribute name="OCTOPART_URL" value="https://octopart.com/max3232cse%2B-maxim+integrated-39430845?r=sp" x="34.671" y="34.671" size="1.778" layer="27" rot="R90" display="off"/>
 <attribute name="OC_FARNELL" value="9725490" x="34.671" y="34.671" size="1.778" layer="27" rot="R90" display="off"/>
 <attribute name="OC_NEWARK" value="90C2890" x="34.671" y="34.671" size="1.778" layer="27" rot="R90" display="off"/>
@@
 </element>
 <element name="JP1" library="Hexabitz" package="1X05/90" package3d_urn="urn:adsk.eagle:package:22467/2" value="" x="34.671" y="48.895" smashed="yes">
+<attribute name="DESCRIPTION" value="Conn Header R/a 5POS 2.54MM MALE" x="34.671" y="48.895" size="1.778" layer="27" display="off"/>
+<attribute name="MFN" value="Sullins" x="34.671" y="48.895" size="1.778" layer="27" display="off"/>
+<attribute name="MPN" value="PEC05SBAN" x="34.671" y="48.895" size="1.778" layer="27" display="off"/>
 <attribute name="NAME" x="42.037" y="43.307" size="1.27" layer="25" ratio="10" rot="R90"/>
+<attribute name="OCTOPART_URL" value="https://octopart.com/pec05sban-sullins-264498?r=sp" x="34.671" y="48.895" size="1.778" layer="27" display="off"/>
 <attribute name="POPULARITY" value="9" x="34.671" y="48.895" size="1.778" layer="27" display="off"/>
 <attribute name="VALUE" x="42.926" y="45.085" size="1.27" layer="27" rot="R90"/>
@@
 <contactref element="U1" pad="P$20"/>
 <wire x1="46.101" y1="35.902" x2="46.3324" y2="36.1334" width="0.254" layer="16"/>
-<wire x1="46.3324" y1="36.1334" x2="46.3324" y2="36.576" width="0.254" layer="16"/>
+<wire x1="46.3324" y1="36.1334" x2="46.3324" y2="36.576" width="0.3556" layer="16"/>
 <via x="46.3324" y="36.576" extent="1-16" drill="0.35"/>
 <wire x1="46.3324" y1="36.576" x2="48.5366" y2="36.576" width="0.3556" layer="1"/>
@@
 <wire x1="29.591" y1="31.33" x2="29.757" y2="31.496" width="0.3556" layer="1"/>
 <wire x1="29.757" y1="31.496" x2="31.5976" y2="31.496" width="0.3556" layer="1"/>
-<wire x1="40.132" y1="38.569" x2="44.3394" y2="38.569" width="0.254" layer="1"/>
-<wire x1="44.3394" y1="38.569" x2="46.3324" y2="36.576" width="0.254" layer="1"/>
+<wire x1="40.132" y1="38.569" x2="44.3394" y2="38.569" width="0.3556" layer="1"/>
+<wire x1="44.3394" y1="38.569" x2="46.3324" y2="36.576" width="0.3556" layer="1"/>
 <wire x1="27.559" y1="31.43" x2="27.498" y2="31.369" width="0.254" layer="1"/>
 <wire x1="27.498" y1="31.369" x2="25.527" y2="31.369" width="0.3556" layer="1"/>
@@
 <wire x1="30.607" y1="41.021" x2="26.416" y2="41.021" width="0.254" layer="16"/>
 <wire x1="22.8092" y1="37.4142" x2="22.8092" y2="35.687" width="0.254" layer="16"/>
-<wire x1="22.8092" y1="35.687" x2="22.8092" y2="34.5948" width="0.254" layer="16"/>
+<wire x1="22.8092" y1="35.687" x2="22.8092" y2="34.5948" width="0.3556" layer="16"/>
 <wire x1="26.416" y1="41.021" x2="22.8092" y2="37.4142" width="0.254" layer="16"/>
 <wire x1="22.8092" y1="34.5948" x2="22.8092" y2="35.687" width="0.3556" layer="1"/>
@@
 <wire x1="26.21933125" y1="36.6242" x2="24.511" y2="34.91586875" width="0.254" layer="16"/>
 <wire x1="24.511" y1="32.004" x2="24.511" y2="34.91586875" width="0.254" layer="16"/>
-<wire x1="24.511" y1="32.004" x2="22.86" y2="32.004" width="0.254" layer="16"/>
+<wire x1="24.511" y1="32.004" x2="22.86" y2="32.004" width="0.3556" layer="16"/>
 <wire x1="22.86" y1="32.004" x2="22.8092" y2="32.0548" width="0.254" layer="16"/>
 <wire x1="22.8092" y1="32.0548" x2="24.511" y2="32.0548" width="0.3556" layer="1"/>
